File: electronics/icom-ctcss-board.kicad_sch (KiCad schematic)
At the start: 38 parts, among them J1 J_MIC_IN, J2 J_RADIO_OUT, J3 J_UI_ENCODER, J4 J_UI_LCD, J5 J_BYPASS, J6 J_UI_LEDS, Q1 2N3904RLRAG, U1 Teyleten USB-C 5V/16MHz

Commit message: updates due to parts availability
Parts:
- C1, C2, C4, C5: Assembly (none) -> 100nF 50V X7R 10%; nonpolar; 2.5mm pitch; body max 4x2.6x5.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; Availability checked (none) -> 2026-10-22; MPN (none) -> K104K15X7RF5TL2; Manufacturer (none) -> Vishay; Purchase URL (none) -> https://www.digikey.com/en/products/detail/vishay-beyschlag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; Supplier (none) -> DigiKey; Supplier SKU (none) -> BC1084CT-ND
- C3: Assembly Nonpolar; 5mm pitch; body 7.2x5x10mm -> Nonpolar 1uF 63V 5%; 5mm pitch; maximum body 7.5x5.1x10.1mm; Availability checked (none) -> 2026-10-22; MPN MKS2C041001F00KSSD -> R82DC4100AA60J; Manufacturer WIMA -> KEMET; Purchase URL (none) -> https://www.digikey.com/en/products/detail/kemet/R82DC4100A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; Supplier (none) -> DigiKey; Supplier SKU (none) -> 399-5860-ND
- C6: footprint CTCSS_THT:C_Film4u7_P5_CNC -> CTCSS_THT:C_Film4u7_P15_CNC; Assembly Nonpolar; 5mm pitch; body 7.2x11x18mm -> Nonpolar 4.7uF 63V 5%; 15mm pitch; maximum body 18x7x12.5mm; Availability checked (none) -> 2026-10-22; MPN MKS2C044701O00KSSD -> B32522C0475J000; Manufacturer WIMA -> TDK; Purchase URL (none) -> https://www.digikey.com/en/products/detail/tdk-electronics-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; Supplier (none) -> DigiKey; Supplier SKU (none) -> 495-1131-ND
- J1, J2: Assembly (none) -> 2.54mm single row; 6mm mating post; 3mm solder tail; mark p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; Availability checked (none) -> 2026-10-22; MPN (none) -> 61300811121; Manufacturer (none) -> Wurth Elektronik; Purchase URL (none) -> https://www.digikey.com/en/products/detail/w%C3%BCrth-elekt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; Supplier (none) -> DigiKey; Supplier SKU (none) -> 732-5321-ND
- J3: Assembly (none) -> 2.54mm single row; 6mm mating post; 3mm solder tail; mark p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; Availability checked (none) -> 2026-10-22; MPN (none) -> 61300511121; Manufacturer (none) -> Wurth Elektronik; Purchase URL (none) -> https://www.digikey.com/en/products/detail/w%C3%BCrth-elekt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; Supplier (none) -> DigiKey; Supplier SKU (none) -> 732-5319-ND
- J4, J6: Assembly (none) -> 2.54mm single row; 6mm mating post; 3mm solder tail; mark p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; Availability checked (none) -> 2026-10-22; MPN (none) -> 61300411121; Manufacturer (none) -> Wurth Elektronik; Purchase URL (none) -> https://www.digikey.com/en/products/detail/w%C3%BCrth-elekt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; Supplier (none) -> DigiKey; Supplier SKU (none) -> 732-5317-ND
- J5: Assembly (none) -> 2.54mm single row; 6mm mating post; 3mm solder tail; mark p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; Availability checked (none) -> 2026-10-22; MPN (none) -> 61300211121; Manufacturer (none) -> Wurth Elektronik; Purchase URL (none) -> https://www.digikey.com/en/products/detail/w%C3%BCrth-elekt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; Supplier (none) -> DigiKey; Supplier SKU (none) -> 732-5315-ND
- Q1: value 2N3904RLRAG -> 2N3904TAR; Assembly Factory-formed 2.54mm pitch ONLY; flat face per drawing -> Factory-formed CASE135AR; 2.54mm nominal pitch; 1 E, 2 B, 3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; Availability checked (none) -> 2026-10-22; MPN 2N3904RLRAG -> 2N3904TAR; Purchase URL (none) -> https://www.digikey.com/en/products/detail/onsemi/2N3904TAR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; Supplier (none) -> DigiKey; Supplier SKU (none) -> 2N3904TARCT-ND
- R1, R2: Assembly (none) -> 1% metal film; 3.6x1.6mm max; form axial leads with tool to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; Availability checked (none) -> 2026-10-22; MPN (none) -> MRS16000C3301FCT00; Manufacturer (none) -> Vishay; Purchase URL (none) -> https://www.digikey.com/en/products/detail/vishay-beyschlag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; Supplier (none) -> DigiKey; Supplier SKU (none) -> BC3934CT-ND
- R10: Assembly (none) -> 1% metal film; 3.6x1.6mm max; form axial leads with tool to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; Availability checked (none) -> 2026-10-22; MPN (none) -> MRS16000C4701FCT00; Manufacturer (none) -> Vishay; Purchase URL (none) -> https://www.digikey.com/en/products/detail/vishay-beyschlag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; Supplier (none) -> DigiKey; Supplier SKU (none) -> BC3940CT-ND
- R11, R5: Assembly (none) -> 1% metal film; 3.6x1.6mm max; form axial leads with tool to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; Availability checked (none) -> 2026-10-22; MPN (none) -> MRS16000C1003FCT00; Manufacturer (none) -> Vishay; Purchase URL (none) -> https://www.digikey.com/en/products/detail/vishay-beyschlag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; Supplier (none) -> DigiKey; Supplier SKU (none) -> BC3921CT-ND
- R12, R13, R14, R15, R3, R9: Assembly (none) -> 1% metal film; 3.6x1.6mm max; form axial leads with tool to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; Availability checked (none) -> 2026-10-22; MPN (none) -> MRS16000C1002FCT00; Manufacturer (none) -> Vishay; Purchase URL (none) -> https://www.digikey.com/en/products/detail/vishay-beyschlag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; Supplier (none) -> DigiKey; Supplier SKU (none) -> BC3918CT-ND
- R4, R8: Assembly (none) -> 1% metal film; 3.6x1.6mm max; form axial leads with tool to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; Availability checked (none) -> 2026-10-22; MPN (none) -> MRS16000C1001FCT00; Manufacturer (none) -> Vishay; Purchase URL (none) -> https://www.digikey.com/en/products/detail/vishay-beyschlag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; Supplier (none) -> DigiKey; Supplier SKU (none) -> BC3915CT-ND
- R6, R7: Assembly (none) -> 1% metal film; 3.6x1.6mm max; form axial leads with tool to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; Availability checked (none) -> 2026-10-22; MPN (none) -> MRS16000C3300FCT00; Manufacturer (none) -> Vishay; Purchase URL (none) -> https://www.digikey.com/en/products/detail/vishay-beyschlag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; Supplier (none) -> DigiKey; Supplier SKU (none) -> BC3933CT-ND
- RV1: Availability checked (none) -> 2026-10-22; Purchase URL (none) -> https://www.digikey.com/en/products/detail/bourns-inc/3296W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; Supplier (none) -> DigiKey; Supplier SKU (none) -> 3296W-103LF-ND
- TP1, TP2, TP3, TP4, TP5, TP6, TP7, TP8: Assembly (none) -> Single 0.64mm square test post; 2.54mm body; 1.1mm drilled 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; Availability checked (none) -> 2026-10-22; MPN (none) -> 61300111121; Manufacturer (none) -> Wurth Elektronik; Purchase URL (none) -> https://www.digikey.com/en/products/detail/w%C3%BCrth-elekt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; Supplier (none) -> DigiKey; Supplier SKU (none) -> 732-5314-ND
- U1: Availability checked (none) -> 2026-10-22; Purchase URL (none) -> https://www.amazon.com/dp/B0B6HYLC44; Supplier (none) -> Amazon; Supplier SKU (none) -> B0B6HYLC44
Other:
- note added: "PTT SENSE / DRIVER: default PTT released during reset. Q1 onsemi 2N3904TAR, factory-formed 2.54mm leads; E=1, B=2, C=3. Initial sink target <=5mA; verify actual radio voltage/current and saturation."
- note added: "SUPPLY: +8V directly to U1 RAW; U1 VCC supplies +5V. C4 RAW decoupling; C5 +5V decoupling; C6 4.7uF TDK film, 15mm pitch. C3 1uF KEMET film, 5mm pitch. Both film capacitors nonpolar, 63V."
- note removed: "PTT SENSE / DRIVER: default PTT released during reset. Q1 onsemi 2N3904RLRAG, factory-formed 2.54mm leads; E=1, B=2, C=3. Initial sink target <=5mA; verify actual radio voltage/current and saturation."
- note removed: "SUPPLY: +8V directly to U1 RAW; U1 VCC supplies +5V. C4 RAW decoupling; C5 +5V decoupling; C6 4.7uF film bulk. C3 1uF film coupling. Both WIMA parts are nonpolar, 63V, 5mm lead pitch."
